File: pcb/pcb.kicad_sch (KiCad schematic)
At the start: 35 parts, among them J1 upd_song, J2 select, J3 swd, SW1 menu, U1 ME2108A, U2 XC6206P333MR, U3 STM32F103C6Tx, U4 TDA2822, U5 AT25xxx

Commit message: pcb ok
Parts:
- added J4: buttons, Connector_PinHeader_2.54mm:PinHeader_1x04_P2.54mm_Vertical, symbol Connector_Generic:Conn_01x04
Connections:
- net +3.3V: now also R22.1
- net +5V: no longer R22.1
- net GND: now also J4.1 (Pin_1)
- net at SW1.2: now also U3.10 (PA0); no longer U3.25 (PB12)
- net at U3.16 (PA6), U5.2 (MISO): now also U3.20 (PB2)
- net at U3.2 (PC13): now also J4.3 (Pin_3)
- net at U3.3 (PC14): now also J4.2 (Pin_2)
- net at U3.4 (PC15): now also J4.4 (Pin_4)
- no-connect marks 21 -> 17
Other:
- moved on the sheet: R22
